Commit message: reworked everything manually, removed wheel joints for visualiuation, reworked scales

File: urdf/vario700_sensorrig.urdf (robot description, URDF)
Before this commit: robot vario700_sensorrig, 15 links, 14 joints
Links:
- removed link OS0_REV6_128_20hz___1024_resolution
- removed link OS0_REV7_128_10hz___512_resolution
- added link os_sensor; visual cylinder length=0.1 radius=0.05
- link Camera_BL: geometry visual box size=0.05 0.05 0.05
- link Camera_BR: geometry visual box size=0.05 0.05 0.05
- link Camera_FL: geometry visual box size=0.05 0.05 0.05
- link Camera_FR: geometry visual box size=0.05 0.05 0.05
- link Camera_ML: geometry visual box size=0.05 0.05 0.05
- link Camera_MR: geometry visual box size=0.05 0.05 0.05
- link back_left_wheel: mass 0.000001 -> 1.0; geometry collision mesh filename=package://vario700_sensorrig/meshes/back_left_wheel_collisi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 scale=.1 .1 .1; visual mesh filename=package://vario700_sensorrig/meshes/back_left_wheel_visuals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 scale=.1 .1 .1
- link back_right_wheel: mass 0.000001 -> 1.0; geometry collision mesh filename=package://vario700_sensorrig/meshes/back_right_wheel_collis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 scale=.1 .1 .1; visual mesh filename=package://vario700_sensorrig/meshes/back_right_wheel_visual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 scale=.1 .1 .1
- link base_link: mass None -> 10.0; geometry collision mesh filename=package://vario700_sensorrig/meshes/base_link_collisions.obj scale=.1 .1 .1; visual mesh filename=package://vario700_sensorrig/meshes/base_link_visuals.obj scale=.1 .1 .1
- link front_left_wheel: mass 0.000001 -> 1.0; geometry collision mesh filename=package://vario700_sensorrig/meshes/front_left_wheel_collis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 scale=.1 .1 .1; visual mesh filename=package://vario700_sensorrig/meshes/front_left_wheel_visual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 scale=.1 .1 .1
- link front_right_wheel: mass 0.000001 -> 1.0; geometry collision mesh filename=package://vario700_sensorrig/meshes/front_right_wheel_colli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 scale=.1 .1 .1; visual mesh filename=package://vario700_sensorrig/meshes/front_right_wheel_visua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 scale=.1 .1 .1
- link sensorrig: mass 0.000001 -> 2.0; geometry collision mesh filename=package://vario700_sensorrig/meshes/sensorrig_collisions.obj scale=.001 .001 .001; visual mesh filename=package://vario700_sensorrig/meshes/sensorrig_visuals.obj scale=.001 .001 .001
Joints:
- removed joint joint_sensorrig-OS0_REV6_128_20hz___1024_resolution
- removed joint joint_sensorrig-OS0_REV7_128_10hz___512_resolution
- added joint joint_sensorrig-os_sensor: type fixed, parent sensorrig, child os_sensor, origin xyz=16.107047 -.000002168 .30456617  rpy=0.0698132 0.7853982 0. 
- joint back_left_joint: axis 1. 0. 0. -> (none); origin xyz=-9.29712 -10.5215 7.9196  rpy=0. 0. 3.1415927 -> xyz=-.929712 -1.05215 .79196  rpy=0. 0. 3.1415927; type continuous -> fixed
- joint back_right_joint: axis 1. 0. 0. -> (none); origin xyz=9.29712 -10.5215 7.9196  rpy=0. 0. 3.1415927 -> xyz=.929712 -1.05215 .79196  rpy=0. 0. 3.1415927; type continuous -> fixed
- joint front_left_joint: axis 1. 0. 0. -> (none); origin xyz=-9.34094 17.2967 5.81455 rpy=0. 0. 3.1415927 -> xyz=-.934094 1.72967 .581455 rpy=0. 0. 3.1415927; type continuous -> fixed
- joint front_right_joint: axis 1. 0. 0. -> (none); origin xyz=9.34094 17.2967 5.81455 rpy=0. 0. 3.1415927 -> xyz=.934094 1.72967 .581455 rpy=0. 0. 3.1415927; type continuous -> fixed
- joint joint_sensorrig-Camera_BL: origin xyz=186.38379 740.865 0.  rpy=1.5707964 0. 0.6981317 -> xyz=18.638379 74.0865 .0  rpy=1.5707964 0. 0.6981317
- joint joint_sensorrig-Camera_BR: origin xyz=186.38379 -740.865 0.  rpy=1.5707964 0. 2.443461  -> xyz=18.638379 -74.0865 .0  rpy=1.5707964 0. 2.443461 
- joint joint_sensorrig-Camera_FL: origin xyz=1394.0425 792.4227 0.  rpy=1.5707964 0. -0.6981317 -> xyz=139.40425 79.24227 .0  rpy=1.5707964 0. -0.6981317
- joint joint_sensorrig-Camera_FR: origin xyz=1394.0425 -792.4227 0.  rpy=1.5707964 0. -2.443461  -> xyz=139.40425 -79.24227 .0  rpy=1.5707964 0. -2.443461 
- joint joint_sensorrig-Camera_ML: origin xyz=785.1372 841.4958 0.  rpy=1.5707964 0. 0.  -> xyz=78.51372 84.14958 .0  rpy=1.5707964 0. 0. 
- joint joint_sensorrig-Camera_MR: origin xyz=785.1372 -841.4958 0.  rpy=1.5707964 0. -3.1415927 -> xyz=78.51372 -84.14958 .0  rpy=1.5707964 0. -3.1415927
- joint sensorrig_joint: origin xyz=0. -13.5969 28.9559 rpy=0. 0. 1.5707964 -> xyz=.0 -1.35969 2.89559 rpy=0. 0. 1.5707964

Commit message: Added rviz file for default visualization; reworked camera joint transforms to match model

File: urdf/vario700_sensorrig.urdf (robot description, URDF)
Before this commit: robot vario700_sensorrig, 14 links, 13 joints
Links:
- removed link Camera_BL
- removed link Camera_BR
- removed link Camera_FL
- removed link Camera_FR
- removed link Camera_ML
- removed link Camera_MR
- added link camera/rear_left; visual box size=0.05 0.05 0.05
- added link camera/rear_mid; visual box size=0.05 0.05 0.05
- added link camera/rear_right; visual box size=0.05 0.05 0.05
- added link camera/side_left; visual box size=0.05 0.05 0.05
- added link camera/side_right; visual box size=0.05 0.05 0.05
Joints:
- removed joint joint_sensorrig-Camera_BL
- removed joint joint_sensorrig-Camera_BR
- removed joint joint_sensorrig-Camera_FL
- removed joint joint_sensorrig-Camera_FR
- removed joint joint_sensorrig-Camera_ML
- removed joint joint_sensorrig-Camera_MR
- added joint joint_sensorrig-camera/rear_left: type fixed, parent sensorrig, child camera/rear_left, origin xyz=.18638379 .740865 .0  rpy=1.5707964 0. 0.6981317
- added joint joint_sensorrig-camera/rear_mid: type fixed, parent sensorrig, child camera/rear_mid, origin xyz=.18638379 .0 .0  rpy=1.5707964 0. 2.443461 
- added joint joint_sensorrig-camera/rear_right: type fixed, parent sensorrig, child camera/rear_right, origin xyz=.18638379 -.740865 .0  rpy=1.5707964 0. 2.443461 
- added joint joint_sensorrig-camera/side_left: type fixed, parent sensorrig, child camera/side_left, origin xyz=.7851372 .8414958 .0  rpy=1.5707964 0. 0. 
- added joint joint_sensorrig-camera/side_right: type fixed, parent sensorrig, child camera/side_right, origin xyz=.7851372 -.8414958 .0  rpy=1.5707964 0. -3.1415927
- joint joint_sensorrig-os_sensor: origin xyz=16.107047 -.000002168 .30456617  rpy=0.0698132 0.7853982 0.  -> xyz=1.6107047 -.000002168 .30456617  rpy=0.0698132 0.7853982 0. 
