Commit message: 0.2.0: add zed_imu_link (additive only)
ZED 2i factory camera-IMU calibration from SDK 5.1.2 as a fixed joint
zed_left_camera_frame -> zed_imu_link, so /zed/zed_node/imu/data has a TF
home with the ROS wrapper's TF publishing disabled. No existing link,
joint, or value modified.

Co-Authored-By: Claude Fable 5 <noreply@anthropic.com>

File: urdf/vario700_sensorrig.urdf (robot description, URDF)
Before this commit: robot vario700_sensorrig, 19 links, 18 joints
Links:
- added link zed_imu_link
Joints:
- added joint zed_left_frame_to_imu: type fixed, parent zed_left_camera_frame, child zed_imu_link, origin xyz=-0.002 -0.023061 0.000217 rpy=-0.003160 0.003185 -0.000015
