Commit message: Added ChaRuCo mono camera calibration - currently not correct

File: urdf/vario700_sensorrig_msa.urdf (robot description, URDF)
Before this commit: robot vario700_sensorrig, 21 links, 20 joints
Joints:
- removed joint joint_camera_rear_mid-camera_rear_left
- removed joint joint_camera_rear_mid-camera_rear_right
- removed joint joint_camera_rear_mid-camera_side_left
- removed joint joint_camera_rear_mid-camera_side_right
- added joint joint_os_sensor-camera_rear_left: type fixed, parent os_sensor, child camera_rear_left, origin xyz=0.987213 -0.716739 -1.10573 rpy=0.338194 -2.49739 0.754168
- added joint joint_os_sensor-camera_rear_right: type fixed, parent os_sensor, child camera_rear_right, origin xyz=0.979937 0.739726 -1.09765 rpy=0.467141 2.53466 2.30594
- added joint joint_os_sensor-camera_side_left: type fixed, parent os_sensor, child camera_side_left, origin xyz=0.536304 -0.868147 -0.633051 rpy=0.791996 -2.31362 0.0204264
- added joint joint_os_sensor-camera_side_right: type fixed, parent os_sensor, child camera_side_right, origin xyz=0.522142 0.877865 -0.631033 rpy=-2.27836 0.834522 0.0180667
