Commit message: manual registration of zed pointcloud added (frame: zed_left_camera_frame; Other ZED links still missing)

File: urdf/vario700_sensorrig_manual.urdf (robot description, URDF)
Before this commit: robot vario700_sensorrig, 18 links, 17 joints
Joints:
- removed joint zed_imu_link_joint
- removed joint zed_left_camera_frame_joint
- removed joint zed_right_camera_frame_joint
- joint zed_camera_link_joint: child zed_camera_link -> zed_left_camera_frame; origin xyz=0 0 0 rpy=0 0 0 -> xyz=0.08 0.26  3.05 rpy=0.0 0.427851 1.570796; parent os_sensor -> base_link

Commit message: renamed camera links to fit camera_info publisher

File: urdf/vario700_sensorrig_manual.urdf (robot description, URDF)
Before this commit: robot vario700_sensorrig, 18 links, 14 joints
Links:
- removed link camera/rear_left
- removed link camera/rear_mid
- removed link camera/rear_right
- removed link camera/side_left
- removed link camera/side_right
- added link camera_rear_left; visual box size=0.05 0.05 0.05
- added link camera_rear_mid; visual box size=0.05 0.05 0.05
- added link camera_rear_right; visual box size=0.05 0.05 0.05
- added link camera_side_left; visual box size=0.05 0.05 0.05
- added link camera_side_right; visual box size=0.05 0.05 0.05
Joints:
- removed joint joint_os_sensor-camera/rear_left
- removed joint joint_os_sensor-camera/rear_mid
- removed joint joint_os_sensor-camera/rear_right
- removed joint joint_os_sensor-camera/side_left
- removed joint joint_os_sensor-camera/side_right
- added joint joint_os_sensor-camera_rear_left: type fixed, parent os_sensor, child camera_rear_left, origin xyz=0.987213 -0.716739 -1.10573 rpy=0.338194 -2.49739 0.754168
- added joint joint_os_sensor-camera_rear_mid: type fixed, parent os_sensor, child camera_rear_mid, origin xyz=1.08013 0.0128897 -1.15956 rpy=0.188916 -3.11455 1.56053
- added joint joint_os_sensor-camera_rear_right: type fixed, parent os_sensor, child camera_rear_right, origin xyz=0.979937 0.739726 -1.09765 rpy=0.467141 2.53466 2.30594
- added joint joint_os_sensor-camera_side_left: type fixed, parent os_sensor, child camera_side_left, origin xyz=0.536304 -0.868147 -0.633051 rpy=0.791996 -2.31362 0.0204264
- added joint joint_os_sensor-camera_side_right: type fixed, parent os_sensor, child camera_side_right, origin xyz=0.522142 0.877865 -0.631033 rpy=-2.27836 0.834522 0.0180667
- added joint zed_imu_joint: type fixed, parent zed_camera_link, child zed_imu_link, origin xyz=0 0 0 rpy=0 0 0
- added joint zed_left_camera_joint: type fixed, parent zed_camera_link, child zed_left_camera_frame, origin xyz=0 0.06 0 rpy=0 0 0
- added joint zed_right_camera_joint: type fixed, parent zed_camera_link, child zed_right_camera_frame, origin xyz=0 -0.06 0 rpy=0 0 0
- joint zed_camera_link_joint: child zed_left_camera_frame -> zed_camera_link

Commit message: Added blickfeld. Frame_ID in message header wrongly recorder with 'Root'. Added 'Root' frame to urdf no correct transform yet.

File: urdf/vario700_sensorrig_manual.urdf (robot description, URDF)
Before this commit: robot vario700_sensorrig, 18 links, 17 joints
Links:
- added link Root; visual box size=0.05 0.05 0.05
Joints:
- added joint joint_os_sensor-blickfeld: type fixed, parent os_sensor, child Root, origin xyz=1.08013 0.0128897 -1.15956 rpy=0.188916 -3.11455 1.56053

Commit message: small syntax error

File: urdf/vario700_sensorrig_manual.urdf (robot description, URDF)
Before this commit: robot vario700_sensorrig, 19 links, 18 joints
Links:
- added link zed_left_camera_optical_frame
Joints:
- added joint zed_left_camera_optical_frame_joint: type fixed, parent zed_left_camera_frame, child zed_left_camera_optical_frame, origin xyz=0 0 0 rpy=-1.57079632679 0 -1.57079632679

Commit message: Did ICP registration for ZED & Ouster Pointcloud, added to urdf.

File: urdf/vario700_sensorrig_manual.urdf (robot description, URDF)
Before this commit: robot vario700_sensorrig, 20 links, 19 joints
Joints:
- removed joint zed_camera_link_joint
- removed joint zed_right_camera_joint
- joint zed_left_camera_joint: origin xyz=0 0.06 0 rpy=0 0 0 -> xyz=-0.017881 -0.118638 0.062218 rpy=-0.015401 -0.354727 -3.119028; parent zed_camera_link -> os_sensor

Commit message: forgot to comment old zed links

File: urdf/vario700_sensorrig_manual.urdf (robot description, URDF)
Before this commit: robot vario700_sensorrig, 20 links, 17 joints
Links:
- removed link zed_camera_link
- removed link zed_imu_link
- removed link zed_right_camera_frame
Joints:
- removed joint zed_imu_joint

Commit message: Added correct ZED frame transforms for right camera and center; ouster IMU transform

File: urdf/vario700_sensorrig_manual.urdf (robot description, URDF)
Before this commit: robot vario700_sensorrig, 17 links, 16 joints
Links:
- removed link os_sensor_imu
- added link os_imu
- added link zed_camera_center
- added link zed_camera_link
- added link zed_right_camera_frame
- added link zed_right_camera_optical_frame
- link zed_left_camera_frame: geometry 
Joints:
- removed joint os_sensor_imu_joint
- added joint os_imu_joint: type fixed, parent os_sensor, child os_imu, origin xyz=-0.002441 -0.009725 0.007533 rpy=0 0 0
- added joint zed_camera_center_joint: type fixed, parent zed_left_camera_frame, child zed_camera_center, origin xyz=0.010 -0.060 0.000 rpy=0 0 0
- added joint zed_camera_link_joint: type fixed, parent zed_camera_center, child zed_camera_link, origin xyz=0 0 -0.015 rpy=0 0 0
- added joint zed_right_camera_joint: type fixed, parent zed_camera_center, child zed_right_camera_frame, origin xyz=-0.010 -0.060 0.000 rpy=0 0 0
- added joint zed_right_camera_optical_frame_joint: type fixed, parent zed_right_camera_frame, child zed_right_camera_optical_frame, origin xyz=0 0 0 rpy=-1.57079632679 0 -1.57079632679
- joint os_sensor_to_os_lidar: origin xyz=0 0 0 rpy=0 0 0 -> xyz=0 0 0.038195 rpy=0 0 0
- joint zed_left_camera_joint: origin xyz=-0.017881 -0.118638 0.062218 rpy=-0.015401 -0.354727 -3.119028 -> xyz=-0.026789 -0.098001 0.035757 rpy=-0.019154 -0.401029 -3.126174

Commit message: Added optical frames for cameras

File: urdf/vario700_sensorrig_manual.urdf (robot description, URDF)
Before this commit: robot vario700_sensorrig, 21 links, 20 joints
Joints:
- joint joint_base_link-os_sensor: origin xyz=0.0 0.26 2.98 rpy=0.0 -0.802851 -1.570796 -> xyz=0.10 0.26 2.98 rpy=0 -0.812851 -1.570796

Commit message: Added charuco board extrinsic params for mono cameras

File: urdf/vario700_sensorrig_manual.urdf (robot description, URDF)
Before this commit: robot vario700_sensorrig, 21 links, 20 joints
Links:
- added link camera_rear_left_optical_frame
- added link camera_rear_mid_optical_frame
- added link camera_rear_right_optical_frame
- added link camera_side_left_optical_frame
- added link camera_side_right_optical_frame
Joints:
- removed joint joint_camera_rear_mid-camera_rear_left
- removed joint joint_camera_rear_mid-camera_side_left
- removed joint joint_camera_rear_mid-camera_side_right
- removed joint joint_os_sensor-camera_rear_mid
- added joint camera_rear_left_optical_joint: type fixed, parent camera_rear_left, child camera_rear_left_optical_frame, origin xyz=0 0 0 rpy=-1.5707963 0 -1.5707963
- added joint camera_rear_mid_optical_joint: type fixed, parent camera_rear_mid, child camera_rear_mid_optical_frame, origin xyz=0 0 0 rpy=-1.5707963 0 -1.5707963
- added joint camera_rear_right_optical_joint: type fixed, parent camera_rear_right, child camera_rear_right_optical_frame, origin xyz=0 0 0 rpy=-1.5707963 0 -1.5707963
- added joint camera_side_left_optical_joint: type fixed, parent camera_side_left, child camera_side_left_optical_frame, origin xyz=0 0 0 rpy=-1.5707963 0 -1.5707963
- added joint camera_side_right_optical_joint: type fixed, parent camera_side_right, child camera_side_right_optical_frame, origin xyz=0 0 0 rpy=-1.5707963 0 -1.5707963
- added joint joint_camera_rear_left-camera_rear_mid: type fixed, parent camera_rear_left, child camera_rear_mid, origin xyz=0.729568 0.078662 -0.036759 rpy=0.185558 0.701033 0.726936
- added joint joint_camera_rear_left-camera_side_left: type fixed, parent camera_rear_left, child camera_side_left, origin xyz=-0.679383 0.060769 -0.066061 rpy=0.188762 -0.343638 -0.366012
- added joint joint_camera_rear_right-camera_side_right: type fixed, parent camera_rear_right, child camera_side_right, origin xyz=0.652059 0.085410 -0.138240 rpy=0.363952 0.463761 0.521473
- added joint joint_os_sensor-camera_rear_left: type fixed, parent os_sensor, child camera_rear_left, origin xyz=0.987213 -0.716739 -1.10573 rpy=0.338194 -2.49739 0.754168
- joint joint_camera_rear_mid-camera_rear_right: origin xyz=-0.421212 -0.541939 -0.303270 rpy=0.509554 0.193946 -0.723323 -> xyz=0.556353 0.283049 -0.436192 rpy=0.257379 0.699633 0.660680

Commit message: Switched back to msa mono camera calibration, added new ICP Calibration from inside garage

File: urdf/vario700_sensorrig_manual.urdf (robot description, URDF)
Before this commit: robot vario700_sensorrig, 26 links, 25 joints
Joints:
- joint joint_camera_rear_left-camera_rear_mid: origin xyz=0.729568 0.078662 -0.036759 rpy=0.185558 0.701033 0.726936 -> xyz=-0.729568 0.078662 -0.036759 rpy=0.185558 -0.701033 -0.726936
- joint os_sensor_to_os_lidar: origin xyz=0 0 0.038195 rpy=0 0 0 -> xyz=0 0 0.038195 rpy=-1.570796 0 0

File: urdf/vario700_sensorrig_msa.urdf (robot description, URDF)
Before this commit: robot vario700_sensorrig, 21 links, 20 joints
Joints:
- joint os_imu_joint: origin xyz=-0.002441 -0.009725 0.007533 rpy=0 0 0 -> xyz=-0.002441 -0.009725 0.007533 rpy=0 -1.570796 0
- joint zed_left_camera_joint: origin xyz=-0.026789 -0.098001 0.035757 rpy=-0.019154 -0.401029 -3.126174 -> xyz=0.166753 -0.157008 -0.192582 rpy=-0.007683 -0.361936 -3.122481
