Commit message: corrected blickfeld lidar position in msa.urdf. Added kalibr-mono-camera calibration to new terasse_urdf. Still worse than msa.

File: urdf/vario700_sensorrig_terasse.urdf (robot description, URDF)
Before this commit: robot vario700_sensorrig, 21 links, 20 joints
Joints:
- removed joint joint_camera_rear_mid-Root
- removed joint joint_os_sensor-camera_rear_left
- removed joint joint_os_sensor-camera_rear_mid
- removed joint joint_os_sensor-camera_rear_right
- removed joint joint_os_sensor-camera_side_left
- added joint joint_camera_rear_left-camera_side_left: type fixed, parent camera_rear_left, child camera_side_left, origin xyz=0.6224 0.1106 -0.2244 rpy=-0.2752 0.4740 0.2358
- added joint joint_camera_rear_mid-blickfeld: type fixed, parent camera_rear_mid, child Root, origin xyz=0.0 0.0 0.0 rpy=1.5708 0.0 -1.5708
- added joint joint_camera_rear_mid-camera_rear_left: type fixed, parent camera_rear_mid, child camera_rear_left, origin xyz=0.7371 0.0765 -0.0433 rpy=0.1261 0.7369 0.7252
- added joint joint_camera_rear_right-camera_rear_mid: type fixed, parent camera_rear_right, child camera_rear_mid, origin xyz=0.5371 0.2753 -0.4252 rpy=0.2365 0.7268 0.6693
- added joint joint_camera_side_right-camera_rear_right: type fixed, parent camera_side_right, child camera_rear_right, origin xyz=0.6585 0.0785 -0.1081 rpy=0.3517 0.4557 0.5183

Commit message: reworked chain of terasse calibration - rear mid as base for mono cams; deleted old deprecated urdfs

File: urdf/vario700_sensorrig_terasse.urdf (robot description, URDF)
Before this commit: robot vario700_sensorrig, 21 links, 20 joints
Joints:
- removed joint joint_camera_rear_mid-blickfeld
- removed joint joint_camera_rear_right-camera_rear_mid
- removed joint joint_camera_side_right-camera_rear_right
- removed joint joint_os_sensor-camera_side_right
- added joint joint_camera_rear_mid-Root: type fixed, parent camera_rear_mid, child Root, origin xyz=-0.300000 0.000000 0.000000 rpy=1.232202 0.000000 0.000003
- added joint joint_camera_rear_mid-camera_rear_right: type fixed, parent camera_rear_mid, child camera_rear_right, origin xyz=0.523172 0.268661 -0.413858 rpy=0.235680 0.724619 0.669439
- added joint joint_camera_rear_right-camera_side_right: type fixed, parent camera_rear_right, child camera_side_right, origin xyz=0.638988 0.076748 -0.110640 rpy=0.355863 0.458518 0.519943
- added joint joint_os_sensor-camera_rear_mid: type fixed, parent os_sensor, child camera_rear_mid, origin xyz=1.08013 0.0128897 -1.15956 rpy=0.188916 -3.11455 1.56053
- joint joint_camera_rear_left-camera_side_left: origin xyz=0.6224 0.1106 -0.2244 rpy=-0.2752 0.4740 0.2358 -> xyz=-0.644967 0.058172 -0.072273 rpy=0.404639 -0.374995 -0.380611
- joint joint_camera_rear_mid-camera_rear_left: origin xyz=0.7371 0.0765 -0.0433 rpy=0.1261 0.7369 0.7252 -> xyz=-0.478852 0.248122 -0.487512 rpy=0.128755 -0.782506 -0.627309

Commit message: terasse calibration now also correct

File: urdf/vario700_sensorrig_terasse.urdf (robot description, URDF)
Before this commit: robot vario700_sensorrig, 21 links, 20 joints
Joints:
- joint joint_camera_rear_left-camera_side_left: origin xyz=-0.644967 0.058172 -0.072273 rpy=0.404639 -0.374995 -0.380611 -> xyz=0.603779435740509 0.107615370836158 -0.220133541697209 rpy=-0.274021914012596 0.476695080303784 0.235842064594591
- joint joint_camera_rear_mid-camera_rear_left: origin xyz=-0.478852 0.248122 -0.487512 rpy=0.128755 -0.782506 -0.627309 -> xyz=0.722 0.076 -0.040 rpy=0.411 0.696 0.725
- joint joint_camera_rear_mid-camera_rear_right: origin xyz=0.523172 0.268661 -0.413858 rpy=0.235680 0.724619 0.669439 -> xyz=-0.706334753202191 0.093880879447860 -0.097177067544477 rpy=0.289483560633349 -0.708003013226559 -0.687384588595347
- joint joint_camera_rear_right-camera_side_right: origin xyz=0.638988 0.076748 -0.110640 rpy=0.355863 0.458518 0.519943 -> xyz=-0.580428993498309 0.178316121505517 -0.240298356120014 rpy=-0.113989203132654 -0.562324884121995 -0.403106074270324

Commit message: changed rear_mids parent to base_link

File: urdf/vario700_sensorrig_terasse.urdf (robot description, URDF)
Before this commit: robot vario700_sensorrig, 21 links, 20 joints
Joints:
- removed joint joint_os_sensor-camera_rear_mid
- added joint joint_base_link-camera_rear_mid: type fixed, parent base_link, child camera_rear_mid, origin xyz=0.113 -1.325 2.967 rpy=-2.140 -0.011 3.115
