Commit message: Added an improved icp calibraiton to kalibr

File: urdf/vario700_sensorrig_kalibr.urdf (robot description, URDF)
Before this commit: robot vario700_sensorrig, 21 links, 20 joints
Joints:
- joint zed_left_camera_joint: origin xyz=0.166753 -0.157008 -0.192582 rpy=-0.007683 -0.361936 -3.122481 -> xyz=0.0 -0.157008 -0.192582 rpy=0.017882 -0.299944 3.103137
