Commit message: Added new MSA Calibration! Minor tweeks in manual kalibr calibration

File: urdf/vario700_sensorrig_msa_new.urdf (robot description, URDF)
Before this commit: robot vario700_sensorrig, 21 links, 20 joints
Links:
- added link novatel_oem7
Joints:
- removed joint joint_base_link-camera_rear_mid
- removed joint joint_camera_rear_left-camera_side_left
- removed joint joint_camera_rear_mid-camera_rear_left
- removed joint joint_camera_rear_mid-camera_rear_right
- removed joint joint_camera_rear_right-camera_side_right
- added joint joint_os_sensor-camera_rear_left: type fixed, parent os_lidar, child camera_rear_left, origin xyz=0.992307 -0.723447 -1.10403 rpy=0.354237 -2.51376 0.741413
- added joint joint_os_sensor-camera_rear_mid: type fixed, parent os_lidar, child camera_rear_mid, origin xyz=1.07908 0.0087477 -1.15012 rpy=0.137981 -3.11007 1.5561
- added joint joint_os_sensor-camera_rear_right: type fixed, parent os_lidar, child camera_rear_right, origin xyz=0.979937 0.739726 -1.09765 rpy=0.467141 2.53466 2.30594
- added joint joint_os_sensor-camera_side_left: type fixed, parent os_lidar, child camera_side_left, origin xyz=0.524944 -0.891771 -0.651685 rpy=0.673336 -2.32848 0.0911685
- added joint joint_os_sensor-camera_side_right: type fixed, parent os_lidar, child camera_side_right, origin xyz=0.518363 0.859965 -0.646625 rpy=-2.3938 0.819432 0.0221712
- added joint novatel_oem7_joint: type fixed, parent os_lidar, child novatel_oem7, origin xyz=-1.79252 -0.0301837 -2.16294 rpy=0.0624273 0.718659 0.0823612
- joint zed_left_camera_joint: origin xyz=0.686738 -0.557055 -0.392554  rpy=0.017882 -0.299944 3.103137 -> xyz=0 0 0 rpy=1.57079632679 0 1.57079632679; parent os_sensor -> zed_left_camera_optical_frame
- joint zed_left_camera_optical_frame_joint: origin xyz=0 0 0 rpy=-1.57079632679 0 -1.57079632679 -> xyz=-0.0768204 -0.0578382 0.135811 rpy=-1.29245 0.0090095 1.55662; parent zed_left_camera_frame -> os_lidar

Commit message: Add surround camera optical frames

File: urdf/vario700_sensorrig_msa_new.urdf (robot description, URDF)
Before this commit: robot vario700_sensorrig, 22 links, 21 joints
Links:
- added link camera_rear_left_optical_frame
- added link camera_rear_mid_optical_frame
- added link camera_rear_right_optical_frame
- added link camera_side_left_optical_frame
- added link camera_side_right_optical_frame
Joints:
- added joint camera_rear_left_optical_frame_joint: type fixed, parent camera_rear_left, child camera_rear_left_optical_frame, origin xyz=0 0 0 rpy=-1.57079632679 0 -1.57079632679
- added joint camera_rear_mid_optical_frame_joint: type fixed, parent camera_rear_mid, child camera_rear_mid_optical_frame, origin xyz=0 0 0 rpy=-1.57079632679 0 -1.57079632679
- added joint camera_rear_right_optical_frame_joint: type fixed, parent camera_rear_right, child camera_rear_right_optical_frame, origin xyz=0 0 0 rpy=-1.57079632679 0 -1.57079632679
- added joint camera_side_left_optical_frame_joint: type fixed, parent camera_side_left, child camera_side_left_optical_frame, origin xyz=0 0 0 rpy=-1.57079632679 0 -1.57079632679
- added joint camera_side_right_optical_frame_joint: type fixed, parent camera_side_right, child camera_side_right_optical_frame, origin xyz=0 0 0 rpy=-1.57079632679 0 -1.57079632679
